File: Thermocouple Gauge/Thermocouple Gauge.kicad_pcb (KiCad board)
At the start: 2 copper layers, 69.2 x 53.3 mm, 13 parts, among them J1 Conn_01x04, J2 Conn_01x20, J3 Conn_01x20, J4 Conn_01x02, J5 Conn_01x04, U1 TLV2461DBV

Commit message: Add files via upload
Connections:
- U1 pad 3: GND -> Net-(R1-Pad2)
- U1 pad 4: Net-(R1-Pad2) -> GND
Routing:
- net Net-(J1-Pad2): track 41.0 -> 11.3 mm
- net Net-(R1-Pad2): track 10.7 -> 9.36 mm
- net GND: track 22.6 -> 23.5 mm, vias 6 -> 7
Other:
- board text added: "HTR 2,3"
- board text added: "SNS 1,4"
- board text added: "Vacuum Thermocouple Gauge Board Rev. 3"
- board text removed: "Vacuum Thermocouple Gauge Board Rev. 2"
