File: Thermocouple Gauge/Thermocouple Gauge.sch (KiCad schematic (older format))
At the start: 10 parts, among them J1 Conn_01x04, J2 Conn_01x20, J3 Conn_01x20, J4 Conn_01x02, J5 Conn_01x04, U1 TLV2461DBV

Commit message: Add files via upload
Connections:
- net GND: now also U1.4 (-); no longer U1.3 (+)
- net at R1.2, R2.1: now also U1.3 (+); no longer U1.4 (-)
Changed lines of the file:
@@
 Wire Wire Line
 	6000 2250 6200 2250
-$Comp
-L power:GND #PWR0101
-U 1 1 5F1D5358
-P 5600 3050
-F 0 "#PWR0101" H 5600 2800 50  0001 C CNN
-F 1 "GND" H 5605 2877 50  0000 C CNN
-F 2 "" H 5600 3050 50  0001 C CNN
-F 3 "" H 5600 3050 50  0001 C CNN
-	1    5600 3050
-	-1   0    0    1
-$EndComp
 Text Notes 7500 4550 0    50   ~ 0
 TI Tiva Launchpad\n
@@
 	9050 4700 9550 4700
 NoConn ~ 7250 2750
-Wire Wire Line
-	5500 3050 5500 3250
-Wire Wire Line
-	5500 3250 5600 3250
-Connection ~ 5500 3050
 $Comp
 L Device:R_POT RV1
@@
 Wire Wire Line
 	6500 2850 5800 2850
+Wire Wire Line
+	5500 3050 5600 3050
+Connection ~ 5500 3050
+$Comp
+L power:GND #PWR?
+U 1 1 60977A0C
+P 5600 3250
+F 0 "#PWR?" H 5600 3000 50  0001 C CNN
+F 1 "GND" H 5605 3077 50  0000 C CNN
+F 2 "" H 5600 3250 50  0001 C CNN
+F 3 "" H 5600 3250 50  0001 C CNN
+	1    5600 3250
+	1    0    0    -1
+$EndComp
 $EndSCHEMATC
